Commit message: Cleaning hand motion

File: model/Hand/hand.URDF (robot description, URDF)
Before this commit: robot hand, 23 links, 22 joints
Joints:
- joint joint10_3: limit lower=-0.88 upper=0.88 effort=10 velocity=1 -> lower=-0.88 upper=0.0 effort=10 velocity=1
- joint joint5: origin xyz=-0.000099998 -0.0016 0.014 rpy=0.174533 0 0 -> xyz=-0.000099998 -0.0016 0.014 rpy=0 0 0

File: model/Hand/index.URDF (robot description, URDF)
Before this commit: robot hand, 11 links, 10 joints
Links:
- removed link thumbp1_c_1
- removed link thumbp1_c_2
- removed link thumbp1_c_3
- removed link thumbp2_c_1
- removed link thumbp2_c_2
- removed link thumbp2_c_3
- removed link thumbp3_c
- removed link thumbp4_c
- removed link thumbp5_c
- removed link thumbp6_c
- added link indexp1_c_1, mass 0.5
- added link indexp1_c_2, mass 0.5
- added link indexp1_c_3, mass 0.5; visual cylinder length=0.005 radius=0.005
- added link indexp2_c, mass 0.5; visual cylinder length=0.005 radius=0.005
- added link indexp3_c, mass 0.5; visual cylinder length=0.005 radius=0.005
- added link indexp4_c, mass 0.5; visual cylinder length=0.005 radius=0.005
- added link indexp5_c, mass 0.5; visual cylinder length=0.005 radius=0.005
Joints:
- removed joint joint2_1
- removed joint joint2_2
- removed joint joint2_3
- removed joint joint6
- added joint joint2: type revolute, parent indexp1_c_3, child indexp2_c, origin xyz=-0.000099998 0.014 -0.0016 rpy=0 0 0, axis 1 0 0, limit lower=-1.57 upper=0.17 effort=10 velocity=1
- joint joint1_1: child thumbp1_c_1 -> indexp1_c_1; origin xyz=0 0 0 rpy=0 -0.191986 0 -> xyz=0 0 0 rpy=-0.0028797933 0 0
- joint joint1_2: child thumbp1_c_2 -> indexp1_c_2; origin xyz=0 0 0 rpy=0 0 -0.083339472 -> xyz=0 0 0 rpy=0 -0.04258603 0; parent thumbp1_c_1 -> indexp1_c_1
- joint joint1_3: axis 1 0 0 -> 0 0 1; child thumbp1_c_3 -> indexp1_c_3; limit lower=-0.785 upper=0 effort=10 velocity=1 -> lower=-0.27 upper=0.27 effort=10 velocity=1; parent thumbp1_c_2 -> indexp1_c_2
- joint joint3: axis 0 1 0 -> 1 0 0; child thumbp3_c -> indexp3_c; limit lower=-0.70 upper=0.27 effort=10 velocity=1 -> lower=-2.10 upper=0 effort=10 velocity=1; origin xyz=-0.0034515 0 0.0204197 rpy=0 0 0 -> xyz=0 0.048 0.00199797 rpy=0 0 0; parent thumbp2_c_3 -> indexp2_c
- joint joint4: axis 0 1 0 -> 1 0 0; child thumbp4_c -> indexp4_c; limit lower=-0 upper=1.57 effort=10 velocity=1 -> lower=-0.875 upper=0 effort=10 velocity=1; origin xyz=-0.0012 0 0.040 rpy=0 0 0 -> xyz=0 0.0279039 0.000899992 rpy=0 0 0; parent thumbp3_c -> indexp3_c
- joint joint5: axis 0 1 0 -> 0 0 0; child thumbp5_c -> indexp5_c; limit lower=-0.90 upper=1.22 effort=10 velocity=1 -> lower=-3.14 upper=3.14 effort=10 velocity=1; origin xyz=-0.0072 0 0.036 rpy=0 0 0 -> xyz=-0.000036879 0.02221986 -0.000910405 rpy=0 0 0; parent thumbp4_c -> indexp4_c; type revolute -> fixed

File: model/myArm750/myArm750.URDF (robot description, URDF)
Before this commit: robot myArm750, 7 links, 6 joints
Links:
- added link meta1_c_1, mass 0.5
- added link meta1_c_2, mass 0.5
- added link meta1_c_3, mass 0.5; visual cylinder length=0.032 radius=0.005
- added link meta2_c, mass 0.5; visual cylinder length=0.016 radius=0.01
- added link wrist, mass 0.5; visual cylinder length=0.016 radius=0.0125
- link base_link: geometry visual cylinder length=0.107 radius=0.03
- link link1: geometry visual cylinder length=0.0669 radius=0.0275
- link link2: geometry visual cylinder length=0.303 radius=0.025
- link link3: geometry visual cylinder length=0.08253 radius=0.0225
- link link4: geometry visual cylinder length=0.24538 radius=0.020
- link link5: geometry visual cylinder length=0.079 radius=0.0175
- link link6: geometry visual cylinder length=0.048 radius=0.015
Joints:
- added joint joint7: type revolute, parent link6, child wrist, origin xyz=0 0.048 0 rpy=0 0 0, axis 0 0 1, limit lower=-0.40 upper=0.40 effort=10 velocity=1
- added joint joint8: type revolute, parent wrist, child meta2_c, origin xyz=0.0011 0.0326447 -0.0025 rpy=0 0 0, axis 1 0 0, limit lower=-1.57 upper=1.57 effort=10 velocity=1
- added joint joint9_1: type fixed, parent meta2_c, child meta1_c_1, origin xyz=-0.0096137 0.0489203 -0.00165902 rpy=0.002443461 0 0, axis 0 0 0, limit lower=-3.14 upper=3.14 effort=10 velocity=1
- added joint joint9_2: type fixed, parent meta1_c_1, child meta1_c_2, origin xyz=0 0 0 rpy=0 0 0.06021386, axis 0 0 0, limit lower=-3.14 upper=3.14 effort=10 velocity=1
- added joint joint9_3: type revolute, parent meta1_c_2, child meta1_c_3, origin xyz=0 0 0 rpy=0 0 0, axis 0 1 0, limit lower=-0.08 upper=0.08 effort=10 velocity=1
- joint joint1: limit lower=-3.14 upper=3.14 effort=10 velocity=1 -> lower=-1.57 upper=1.57 effort=10 velocity=1
- joint joint2: limit lower=-3.14 upper=3.14 effort=10 velocity=1 -> lower=-1.57 upper=1.57 effort=10 velocity=1
- joint joint3: limit lower=-3.14 upper=3.14 effort=10 velocity=1 -> lower=-1.57 upper=1.57 effort=10 velocity=1
- joint joint4: limit lower=-3.14 upper=3.14 effort=10 velocity=1 -> lower=-1.57 upper=1.57 effort=10 velocity=1
- joint joint5: limit lower=-3.14 upper=3.14 effort=10 velocity=1 -> lower=-1.57 upper=1.57 effort=10 velocity=1
- joint joint6: limit lower=-3.14 upper=3.14 effort=10 velocity=1 -> lower=-1.57 upper=1.57 effort=10 velocity=1
